File: controller.kicad_pcb (KiCad board)
At the start: 2 copper layers, 26 parts, among them J1 CONN_01X04, J2 CONN_01X02, J3 CONN_01X02, J4 CONN_01X02, J5 CONN_01X02, J6 CONN_01X02, U1 ATTINY13A-SU

Commit message: save changes
Parts:
- removed J5, J6: CONN_01X02, Connectors:PINHEAD1-2
- added C7: 0.1u, Capacitors_SMD:C_0805, F.Cu at (212.6, 39.1)
- added C8: 220u, Capacitors_SMD:CP_Elec_6.3x7.7, F.Cu at (214.4, 59.4)
- added C9: 470u, Capacitors_Tantalum_SMD:CP_Tantalum_Case-V_EIA-7343-20_Hand, F.Cu at (219.5, 41.7)
- added D4: 5V1, TO_SOT_Packages_SMD:SOT-23, F.Cu at (195.9, 111.7)
- added Q1: AO3401A, TO_SOT_Packages_SMD:SOT-23, F.Cu at (189.8, 111.7)
- added Q2: AO3400A, TO_SOT_Packages_SMD:SOT-23, F.Cu at (110.5, 120.9)
- added R10: 1.5K, Resistors_SMD:R_0805, F.Cu at (200.4, 112.0)
- added R8: 1K, Resistors_SMD:R_0805, F.Cu at (204.7, 112.0)
- added R9: 330, Resistors_SMD:R_0805, F.Cu at (213.9, 44.1)
- C1: value 47uF -> 220u; footprint Capacitors_SMD:CP_Elec_5x5.3 -> Capacitors_SMD:CP_Elec_6.3x7.7
- C2, C5: footprint Capacitors_SMD:C_1210 -> Capacitors_SMD:C_0805
- C4: footprint Capacitors_SMD:CP_Elec_5x5.3 -> Capacitors_SMD:CP_Elec_4x5.7
- C6: value 220uF -> 470u
- D1: value Red -> green
- D2: value Green -> red
- D3: value D_Schottky -> 5A
- J1: value CONN_01X04 -> CONN_01X02; footprint Connectors_Molex:Molex_KK-6410-04_04x2.54mm_Straight -> Connectors_Molex:Molex_KK-6410-02_02x2.54mm_Straight
- J2, J3: footprint Connectors:PINHEAD1-2 -> Connectors_Molex:Molex_KK-6410-02_02x2.54mm_Straight
- J4: value CONN_01X02 -> SPI; footprint Connectors:PINHEAD1-2 -> Connectors_Molex:Molex_KK-6410-03_03x2.54mm_Straight
- R1, R2: value 220 -> 330; footprint Resistors_SMD:R_1206 -> Resistors_SMD:R_0805
- R3: value 220 -> 1M
- R5: value 3.3K -> 3.6K; footprint Resistors_SMD:R_1206 -> Resistors_SMD:R_0805
- R6: value 1K -> 1.2K; footprint Resistors_SMD:R_1206 -> Resistors_SMD:R_0805
- R7: value 10K -> 1K; footprint Resistors_SMD:R_1206 -> Resistors_SMD:R_0805
- U1: value ATTINY13A-SU -> ATTINY24A-SSU; footprint SMD_Packages:SOIC-8-N -> Housings_SOIC:SOIC-14_3.9x8.7mm_Pitch1.27mm
- moved C2 104.7 mm to (55.1, 76.6)
- moved C5 104.7 mm to (90.1, 58.6)
- moved D1 104.7 mm to (115.1, 88.6)
- moved D2 104.7 mm to (115.1, 59.6)
- moved J1 104.7 mm to (111.1, 69.0)
- moved J2 104.7 mm to (95.1, 57.6)
- moved J3 104.7 mm to (62.1, 82.6)
- moved J4 104.7 mm to (111.1, 83.6)
- moved R1 104.7 mm to (110.1, 88.6)
- moved R2 104.7 mm to (100.1, 81.1)
- moved R5 104.7 mm to (91.1, 70.6)
- moved R6 104.7 mm to (67.1, 75.6)
- moved R7 104.7 mm to (105.2, 65.8)
- moved C3 104.7 mm to (97.0, 81.8)
- moved C4 104.7 mm to (96.3, 87.6)
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Connections:
- C1 pad 1: +2V8 -> Net-(C1-Pad1)
- C2 pad 1: +2V8 -> Net-(C1-Pad1)
- DC1 pad 2: Net-(DC1-Pad2) -> EN
- DC1 pad 4: +2V8 -> Net-(C1-Pad1)
- J1 pad 1: /reset -> /ss
- J1 pad 2: /sck -> /rst
- J3 pad 2: +2V8 -> VDD
- J4 pad 1: Net-(D1-Pad2) -> /sck
- J4 pad 2: /mosi -> /miso
- JP1 pad 1: Net-(J6-Pad1) -> Net-(JP1-Pad1)
- L1 pad 2: +2V8 -> Net-(C1-Pad1)
- R2 pad 1: Net-(R2-Pad1) -> Net-(D2-Pad1)
- R2 pad 2: +2V8 -> GND
- R3 pad 1: Net-(D2-Pad1) -> EN
- R4 pad 1: GND -> Net-(JP1-Pad1)
- R4 pad 2: Net-(J6-Pad1) -> GND
- R7 pad 1: GND -> Net-(R7-Pad1)
- R7 pad 2: Net-(DC1-Pad2) -> /pwr_ctrl
- U1 pad 1: /reset -> +2V8
- U1 pad 2: Net-(DC1-Pad2) -> Net-(D1-Pad2)
- U1 pad 3: Net-(R2-Pad1) -> Net-(D2-Pad2)
- U1 pad 4: GND -> /rst
- U1 pad 5: /mosi -> /ss
- U1 pad 6: /miso -> EN
- U1 pad 7: /sck -> /mosi
- U1 pad 8: +2V8 -> /miso
Routing:
- net GND: track 201.5 -> 12.4 mm, vias 1 -> 0
- net +2V8: track 98.1 -> 1.22 mm
- net Net-(DC1-Pad2): track 70.5 -> 0.00 mm, vias 2 -> 0
- net /sck: track 45.3 -> 0.00 mm
- net Net-(DC1-Pad5): track 30.2 -> 0.00 mm
- net +5V: track 28.9 -> 3.11 mm
- net /miso: track 20.7 -> 0.00 mm
- net /reset: track 16.2 -> 0.00 mm
- net Net-(J6-Pad1): track 14.7 -> 0.00 mm
- net /mosi: track 12.3 -> 0.00 mm
- net Net-(D1-Pad2): track 9.36 -> 0.00 mm
- net Net-(D3-Pad2): track 43.5 -> 34.3 mm, vias 1 -> 0
- net Net-(D2-Pad2): track 8.53 -> 0.00 mm
- net EN: track 0.00 -> 6.44 mm
- net Net-(R2-Pad1): track 5.43 -> 0.00 mm
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- removed copper zone on B.Cu, net GND
- removed copper zone on F.Cu, net GND

Commit message: Complete pcb
Parts:
- moved C2 168.8 mm to (223.6, 66.7), turned to 0 degrees
- moved R6 146.0 mm to (212.6, 63.6), turned to 270 degrees
- moved D3 132.7 mm to (217.9, 51.1), turned to 270 degrees
- moved C5 131.9 mm to (221.7, 50.4)
- moved J3 128.8 mm to (183.1, 38.4), turned to 180 degrees
- moved R5 121.9 mm to (212.6, 59.8), turned to 270 degrees
- moved J2 116.8 mm to (211.5, 47.0), turned to 90 degrees
- moved R2 111.1 mm to (208.2, 55.0)
- moved J1 103.6 mm to (210.1, 38.4), turned to 0 degrees
- moved C3 103.1 mm to (196.5, 54.6), turned to 180 degrees
- moved J4 100.1 mm to (200.4, 38.4), turned to 0 degrees
- moved R1 100.0 mm to (204.6, 55.6), turned to 0 degrees
- moved Q2 100.0 mm to (192.3, 63.2)
- moved R4 98.9 mm to (182.6, 63.8)
- moved C4 97.9 mm to (189.4, 56.9)
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Connections:
- net Net-(D1-Pad2) renamed /green
- net Net-(D2-Pad2) renamed /red
Routing:
- net GND: track 12.4 -> 104.1 mm
- net Net-(C1-Pad1): track 0.70 -> 89.3 mm
- net +2V8: track 1.22 -> 48.1 mm
- net EN: track 6.44 -> 44.7 mm, vias 0 -> 2
- net +5V: track 3.11 -> 38.5 mm
- net Net-(JP1-Pad1): track 0.40 -> 24.5 mm, vias 0 -> 1
- net Net-(R7-Pad1): track 0.00 -> 22.3 mm, vias 0 -> 2
- net /rst: track 0.60 -> 19.9 mm
- net Net-(DC1-Pad5): track 0.00 -> 17.9 mm
- net /ss: track 0.30 -> 17.6 mm
- net /sck: track 0.00 -> 16.2 mm
- net /miso: track 0.00 -> 15.6 mm
- net /mosi: track 0.00 -> 11.7 mm
- net Net-(R10-Pad2): track 0.00 -> 11.2 mm
- net /red: track 0.00 -> 8.26 mm
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- added copper zone on B.Cu, net GND
- added copper zone on F.Cu, net GND

Commit message: change pcb
Parts:
- removed C7: 0.1u, Capacitors_SMD:C_0805
- added R11: 0, Resistors_SMD:R_2512, F.Cu at (211.7, 51.3)
- added R12: 0, Resistors_SMD:R_2512, F.Cu at (181.9, 56.1)
- added R13: 0, Resistors_SMD:R_2512, F.Cu at (181.2, 64.8)
- J4: value SPI -> CONN_01X04; footprint Connectors_Molex:Molex_KK-6410-03_03x2.54mm_Straight -> Connectors_Molex:Molex_KK-6410-04_04x2.54mm_Straight
- moved J4 11.9 mm to (188.5, 38.4)
- moved R4 10.9 mm to (187.9, 54.2), turned to 270 degrees
- moved C5 10.5 mm to (213.7, 43.6), turned to 180 degrees
- moved JP1 10.3 mm to (187.6, 48.3)
- moved J2 8.97 mm to (213.9, 38.4), turned to 180 degrees
- moved J1 8.38 mm to (201.7, 38.4)
- moved R7 6.28 mm to (183.0, 60.5)
- moved R8 5.62 mm to (176.4, 53.5), turned to 270 degrees
- moved C4 4.13 mm to (192.3, 59.8), turned to 90 degrees
- moved Q2 3.66 mm to (189.7, 65.9), turned to 90 degrees
- moved R1 3.05 mm to (201.5, 55.6)
- moved R2 2.67 mm to (205.5, 55.6), turned to 180 degrees
- moved D4 2.57 mm to (180.6, 52.3)
- moved L1 2.50 mm to (236.5, 43.7), turned to 0 degrees
- moved R10 2.22 mm to (181.9, 47.8)
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Connections:
- net /pwr_ctrl renamed Net-(Q2-Pad1)
- DC1 pad 2: EN -> Net-(DC1-Pad2)
- J4 pad 1: /sck -> Net-(J4-Pad1)
- J4 pad 2: /miso -> /sck
- J4 pad 3: /mosi -> /miso
- R3 pad 1: EN -> Net-(DC1-Pad2)
- U1 pad 10: Net-(R7-Pad1) -> Net-(J4-Pad1)
- U1 pad 11: Net-(JP1-Pad1) -> Net-(R10-Pad2)
- U1 pad 12: Net-(R10-Pad2) -> Net-(JP1-Pad1)
- U1 pad 13: Net-(C7-Pad2) -> Net-(R7-Pad1)
Routing:
- net GND: track 104.1 -> 16.9 mm
- net Net-(DC1-Pad2): track 0.00 -> 20.4 mm
- net +2V8: track 48.1 -> 29.3 mm
- net EN: track 44.7 -> 30.4 mm, vias 2 -> 0
- net Net-(JP1-Pad1): track 24.5 -> 12.0 mm, vias 1 -> 0
- net Net-(J4-Pad1): track 0.00 -> 10.8 mm
- net /miso: track 15.6 -> 6.34 mm
- net Net-(D3-Pad2): track 37.9 -> 29.0 mm
- net Net-(Q2-Pad1): track 3.52 -> 11.6 mm
- net /sck: track 16.2 -> 8.54 mm
- net /ss: track 17.6 -> 10.8 mm
- net /rst: track 19.9 -> 13.2 mm
- net Net-(R7-Pad1): track 22.3 -> 16.9 mm, vias 2 -> 0
- net Net-(D4-Pad1): track 5.13 -> 0.78 mm
- net /mosi: track 11.7 -> 7.40 mm
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- removed copper zone on B.Cu, net GND
- removed copper zone on F.Cu, net GND

Commit message: Add last changes
Parts:
- removed R12, R13: 0, Resistors_SMD:R_2512
- added JP2: Jumper, Resistors_SMD:R_2512, F.Cu at (181.4, 58.4)
- added JP3: Jumper, Resistors_SMD:R_2512, F.Cu at (181.2, 65.1)
- added JP4: Jumper, Resistors_THT:R_Axial_DIN0204_L3.6mm_D1.6mm_P2.54mm_Vertical, F.Cu at (208.0, 42.4)
- moved R7 4.99 mm to (188.0, 59.7)
- moved R8 2.25 mm to (178.3, 52.3)
- moved D4 1.80 mm to (182.4, 52.6)
- moved DC1 1.27 mm to (230.7, 58.6)
Connections:
- R11 pad 2: EN -> Net-(JP4-Pad2)
Routing:
- net +2V8: track 29.3 -> 50.6 mm
- net Net-(D4-Pad1): track 0.78 -> 9.64 mm
- net EN: track 30.4 -> 23.1 mm
- net GND: track 16.9 -> 23.5 mm
- net Net-(R7-Pad1): track 16.9 -> 22.5 mm
- net Net-(Q2-Pad1): track 11.6 -> 16.8 mm
- net Net-(JP4-Pad2): track 0.00 -> 5.03 mm
- net Net-(DC1-Pad2): track 20.4 -> 22.3 mm
- net Net-(D3-Pad2): track 29.0 -> 30.6 mm
- net Net-(DC1-Pad5): track 17.9 -> 16.6 mm
- net Net-(C1-Pad1): track 86.6 -> 87.6 mm
- added copper zone on F.Cu, net GND
