File: controller.sch (KiCad schematic (older format))
At the start: 35 parts, among them J1 CONN_01X02, J2 CONN_01X02, J3 CONN_01X02, J4 CONN_01X04, Q1 AO3401A, Q2 AO3400A, U1 ATTINY24A-SSU

Commit message: Add last changes
Parts:
- removed R12, R13: 0, Resistors_SMD:R_2512, symbol R
- added JP? (x3): Jumper, symbol Jumper
Connections:
- net +2V8: now also JP?.1, JP?.2
- net EN: now also JP?.1; no longer R11.2
- net GND: now also JP?.1, JP?.2
- new net: JP?.2, R11.2
Changed lines of the file:
@@
 Text Label 4950 2700 0    60   ~ 0
 mosi
-Text GLabel 8350 4950 3    60   Input ~ 0
+Text GLabel 7650 5550 3    60   Input ~ 0
 EN
 Wire Wire Line
@@
 Wire Wire Line
 	2000 2500 2000 2650
-$Comp
-L R R3
-U 1 1 593439D7
-P 8700 4850
-F 0 "R3" H 8770 4896 50  0000 L CNN
-F 1 "1M" H 8770 4805 50  0000 L CNN
-F 2 "Resistors_SMD:R_1206" V 8630 4850 50  0001 C CNN
-F 3 "" H 8700 4850 50  0001 C CNN
-	1    8700 4850
-	1    0    0    -1
-$EndComp
-$Comp
-L GND #PWR21
-U 1 1 59343DED
-P 8700 5200
-F 0 "#PWR21" H 8700 4950 50  0001 C CNN
-F 1 "GND" H 8700 5050 50  0000 C CNN
-F 2 "" H 8700 5200 50  0001 C CNN
-F 3 "" H 8700 5200 50  0001 C CNN
-	1    8700 5200
-	1    0    0    -1
-$EndComp
-Wire Wire Line
-	8700 5000 8700 5200
-Wire Wire Line
-	8700 4700 8700 4500
-Wire Wire Line
-	8700 4500 8350 4500
 Connection ~ 8350 4500
 Wire Wire Line
@@
 Text Label 2350 4750 0    60   ~ 0
 vdd
+Wire Wire Line
+	4950 2100 5050 2100
+Wire Wire Line
+	5450 2300 4950 2300
+Wire Wire Line
+	4950 2200 6850 2200
+Wire Wire Line
+	6900 2300 6850 2300
+$Comp
+L CONN_01X04 J4
+U 1 1 5971243F
+P 5700 2550
+F 0 "J4" H 5778 2591 50  0000 L CNN
+F 1 "CONN_01X04" H 5778 2500 50  0000 L CNN
+F 2 "Connectors_Molex:Molex_KK-6410-04_04x2.54mm_Straight" H 5700 2550 50  0001 C CNN
+F 3 "" H 5700 2550 50  0001 C CNN
+	1    5700 2550
+	1    0    0    -1
+$EndComp
+Wire Wire Line
+	5350 2100 6250 2100
+Wire Wire Line
+	4950 2400 5500 2400
+$Comp
+L GND #PWR15
+U 1 1 59712EF4
+P 6000 1000
+F 0 "#PWR15" H 6000 750 50  0001 C CNN
+F 1 "GND" H 6000 850 50  0000 C CNN
+F 2 "" H 6000 1000 50  0001 C CNN
+F 3 "" H 6000 1000 50  0001 C CNN
+	1    6000 1000
+	1    0    0    -1
+$EndComp
+Wire Wire Line
+	6100 950  6000 950
+Wire Wire Line
+	6000 950  6000 1000
+$Comp
+L GND #PWR?
+U 1 1 597254C7
+P 6750 1050
+F 0 "#PWR?" H 6750 800 50  0001 C CNN
+F 1 "GND" H 6750 900 50  0000 C CNN
+F 2 "" H 6750 1050 50  0001 C CNN
+F 3 "" H 6750 1050 50  0001 C CNN
+	1    6750 1050
+	1    0    0    -1
+$EndComp
+Wire Wire Line
+	6700 950  6750 950
+Wire Wire Line
+	6750 950  6750 1050
+$Comp
+L Jumper JP?
+U 1 1 597252F1
+P 6400 950
+F 0 "JP?" H 6400 1214 50  0000 C CNN
+F 1 "Jumper" H 6400 1123 50  0000 C CNN
+F 2 "" H 6400 950 50  0001 C CNN
+F 3 "" H 6400 950 50  0001 C CNN
+	1    6400 950
+	1    0    0    -1
+$EndComp
+$Comp
+L +2V8 #PWR?
+U 1 1 5972572D
+P 7350 1050
+F 0 "#PWR?" H 7350 900 50  0001 C CNN
+F 1 "+2V8" H 7350 1190 50  0000 C CNN
+F 2 "" H 7350 1050 50  0001 C CNN
+F 3 "" H 7350 1050 50  0001 C CNN
+	1    7350 1050
+	1    0    0    -1
+$EndComp
+$Comp
+L Jumper JP?
+U 1 1 59725809
+P 7700 1150
+F 0 "JP?" H 7700 1414 50  0000 C CNN
+F 1 "Jumper" H 7700 1323 50  0000 C CNN
+F 2 "" H 7700 1150 50  0001 C CNN
+F 3 "" H 7700 1150 50  0001 C CNN
+	1    7700 1150
+	1    0    0    -1
+$EndComp
+Wire Wire Line
+	7350 1050 7350 1150
+Wire Wire Line
+	7350 1150 7400 1150
+$Comp
+L +2V8 #PWR?
+U 1 1 597259A2
+P 8050 1050
+F 0 "#PWR?" H 8050 900 50  0001 C CNN
+F 1 "+2V8" H 8050 1190 50  0000 C CNN
+F 2 "" H 8050 1050 50  0001 C CNN
+F 3 "" H 8050 1050 50  0001 C CNN
+	1    8050 1050
+	1    0    0    -1
+$EndComp
+Wire Wire Line
+	8050 1050 8050 1150
+Wire Wire Line
+	8050 1150 8000 1150
 $Comp
 L R R11
@@
 $EndComp
 Wire Wire Line
-	4950 2100 5050 2100
-Wire Wire Line
-	5450 2300 4950 2300
-Wire Wire Line
-	4950 2200 6850 2200
-Wire Wire Line
-	6900 2300 6850 2300
-$Comp
-L CONN_01X04 J4
-U 1 1 5971243F
-P 5700 2550
-F 0 "J4" H 5778 2591 50  0000 L CNN
-F 1 "CONN_01X04" H 5778 2500 50  0000 L CNN
-F 2 "Connectors_Molex:Molex_KK-6410-04_04x2.54mm_Straight" H 5700 2550 50  0001 C CNN
-F 3 "" H 5700 2550 50  0001 C CNN
-	1    5700 2550
-	1    0    0    -1
-$EndComp
-Wire Wire Line
-	5350 2100 6250 2100
-Wire Wire Line
-	4950 2400 5500 2400
-$Comp
-L R R12
-U 1 1 59712D8F
-P 6600 1300
-F 0 "R12" H 6670 1346 50  0000 L CNN
-F 1 "0" H 6670 1255 50  0000 L CNN
-F 2 "Resistors_SMD:R_2512" V 6530 1300 50  0001 C CNN
-F 3 "" H 6600 1300 50  0001 C CNN
-	1    6600 1300
-	1    0    0    -1
-$EndComp
-$Comp
-L GND #PWR17
-U 1 1 59712E0F
-P 6950 1100
-F 0 "#PWR17" H 6950 850 50  0001 C CNN
-F 1 "GND" H 6950 950 50  0000 C CNN
-F 2 "" H 6950 1100 50  0001 C CNN
-F 3 "" H 6950 1100 50  0001 C CNN
-	1    6950 1100
-	1    0    0    -1
-$EndComp
-Wire Wire Line
-	6600 1150 6600 950
-Wire Wire Line
-	6600 950  6950 950
-Wire Wire Line
-	6950 950  6950 1100
-$Comp
-L GND #PWR15
-U 1 1 59712EF4
-P 6600 1550
-F 0 "#PWR15" H 6600 1300 50  0001 C CNN
-F 1 "GND" H 6600 1400 50  0000 C CNN
-F 2 "" H 6600 1550 50  0001 C CNN
-F 3 "" H 6600 1550 50  0001 C CNN
-	1    6600 1550
-	1    0    0    -1
-$EndComp
-Wire Wire Line
-	6600 1450 6600 1550
-$Comp
-L R R13
-U 1 1 597134B8
-P 7800 1100
-F 0 "R13" H 7870 1146 50  0000 L CNN
-F 1 "0" H 7870 1055 50  0000 L CNN
-F 2 "Resistors_SMD:R_2512" V 7730 1100 50  0001 C CNN
-F 3 "" H 7800 1100 50  0001 C CNN
-	1    7800 1100
-	1    0    0    -1
-$EndComp
-$Comp
-L +2V8 #PWR19
-U 1 1 59713526
-P 7800 950
-F 0 "#PWR19" H 7800 800 50  0001 C CNN
-F 1 "+2V8" H 7800 1090 50  0000 C CNN
-F 2 "" H 7800 950 50  0001 C CNN
-F 3 "" H 7800 950 50  0001 C CNN
-	1    7800 950
-	1    0    0    -1
-$EndComp
-$Comp
-L +2V8 #PWR20
-U 1 1 59713577
-P 8150 1250
-F 0 "#PWR20" H 8150 1100 50  0001 C CNN
-F 1 "+2V8" H 8150 1390 50  0000 C CNN
-F 2 "" H 8150 1250 50  0001 C CNN
-F 3 "" H 8150 1250 50  0001 C CNN
-	1    8150 1250
-	1    0    0    -1
-$EndComp
-Wire Wire Line
-	7800 1250 8150 1250
+	8350 5350 8350 4950
+$Comp
+L GND #PWR21
+U 1 1 59343DED
+P 8700 5200
+F 0 "#PWR21" H 8700 4950 50  0001 C CNN
+F 1 "GND" H 8700 5050 50  0000 C CNN
+F 2 "" H 8700 5200 50  0001 C CNN
+F 3 "" H 8700 5200 50  0001 C CNN
+	1    8700 5200
+	1    0    0    -1
+$EndComp
+Wire Wire Line
+	8700 5000 8700 5200
+Wire Wire Line
+	8700 4500 8350 4500
+Wire Wire Line
+	8700 4700 8700 4500
+$Comp
+L R R3
+U 1 1 593439D7
+P 8700 4850
+F 0 "R3" H 8770 4896 50  0000 L CNN
+F 1 "1M" H 8770 4805 50  0000 L CNN
+F 2 "Resistors_SMD:R_1206" V 8630 4850 50  0001 C CNN
+F 3 "" H 8700 4850 50  0001 C CNN
+	1    8700 4850
+	1    0    0    -1
+$EndComp
+Wire Wire Line
+	7650 5350 7650 5550
+Wire Wire Line
+	8250 5350 8350 5350
+$Comp
+L Jumper JP?
+U 1 1 5973A69E
+P 7950 5350
+F 0 "JP?" H 7950 5614 50  0000 C CNN
+F 1 "Jumper" H 7950 5523 50  0000 C CNN
+F 2 "" H 7950 5350 50  0001 C CNN
+F 3 "" H 7950 5350 50  0001 C CNN
+	1    7950 5350
+	1    0    0    -1
+$EndComp
 $EndSCHEMATC
